File: hardware/gpio.kicad_sch (KiCad schematic)
At the start: 23 parts, among them J2 HDMI_C_1.3, U3 ECP5U_12_CABGA256, U5 PCA9306DC1

Commit message: Last checks
Parts:
- C26: renamed from C44; LCSC Part # (none) -> C19702
- renumbered C45 to C27, C46 to C28, C21 to C29, C22 to C30, C23 to C31, C24 to C32, C25 to C33, C26 to C34, C27 to C35, C28 to C36, C29 to C37, R16 to R12, R17 to R13, R18 to R14, R11 to R15, R12 to R16, R13 to R17, R14 to R18, R15 to R19, U3 to U1
Connections:
- no-connect marks 0 -> 14
