File: hardware/power.kicad_sch (KiCad schematic)
At the start: 38 parts, among them U1 TLV62569DBV, U2 TLV62569DBV, U3 ECP5U_12_CABGA256, U4 TLV62569DBV, Y1 SIT8008xx-1x-xxE-100.000000

Commit message: Final revision
Parts:
- C1, C13, C14, C18, C2, C3: JLCPCB Part # C59461 -> (none); LCSC Part # (none) -> C59461
- C10, C11, C12, C16, C17, C20, C50, C51, C52, C7, C8, C9: JLCPCB Part # C307331 -> (none); LCSC Part # (none) -> C307331
- FB1: JLCPCB Part # C1015 -> (none); LCSC Part # (none) -> C1015
- L1, L2, L3: JLCPCB Part # C1043 -> (none); LCSC Part # (none) -> C1043
- R10: JLCPCB Part # C25890 -> (none); LCSC Part # (none) -> C25890
- R5: JLCPCB Part # C25744 -> (none); LCSC Part # (none) -> C25744
- R6: JLCPCB Part # C25752 -> (none); LCSC Part # (none) -> C25752
- R7, R9: JLCPCB Part # C25756 -> (none); LCSC Part # (none) -> C25756
- R8: JLCPCB Part # C25900 -> (none); LCSC Part # (none) -> C25900
- U1, U2, U4: JLCPCB Part # C141836 -> (none); LCSC Part # (none) -> C141836
- U3: JLCPCB Part # C1521614 -> (none); LCSC Part # (none) -> C1521614
- Y1: value SIT8008xx-1x-xxE-100.000000 -> SITxxxxxx-1x-33E-50.000000; JLCPCB Part # C1182928 -> (none); LCSC Part # (none) -> C1182928
Changed lines of the file:
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@@
 			)
 		)
-		(property "JLCPCB Part #" "C1015"
+		(property "LCSC Part #" "C1015"
 			(at 181.61 71.12 0)
 			(effects
@@
 					(size 1.27 1.27)
 				)
-				(hide yes)
 			)
 		)
@@
 			)
 		)
-		(property "JLCPCB Part #" "C307331 "
+		(property "LCSC Part #" "C307331 "
 			(at 76.2 67.31 0)
 			(effects
@@
 					(size 1.27 1.27)
 				)
-				(hide yes)
 			)
 		)
@@
 			)
 		)
-		(property "JLCPCB Part #" "C25752"
+		(property "LCSC Part #" "C25752"
 			(at 54.61 44.45 0)
 			(effects
@@
 					(size 1.27 1.27)
 				)
-				(hide yes)
 			)
 		)
@@
 			)
 		)
-		(property "JLCPCB Part #" "C307331 "
+		(property "LCSC Part #" "C307331 "
 			(at 198.12 74.93 0)
 			(effects
@@
 					(size 1.27 1.27)
 				)
-				(hide yes)
 			)
 		)
@@
 			)
 		)
-		(property "JLCPCB Part #" "C1043"
+		(property "LCSC Part #" "C1043"
 			(at 49.53 96.52 0)
 			(effects
@@
 					(size 1.27 1.27)
 				)
-				(hide yes)
 			)
 		)
@@
 			)
 		)
-		(property "JLCPCB Part #" "C141836"
+		(property "LCSC Part #" "C141836"
 			(at 36.83 31.75 0)
 			(effects
@@
 					(size 1.27 1.27)
 				)
-				(hide yes)
 			)
 		)
@@
 			)
 		)
-		(property "JLCPCB Part #" "C25756 "
+		(property "LCSC Part #" "C25756 "
 			(at 54.61 101.6 0)
 			(effects
@@
 					(size 1.27 1.27)
 				)
-				(hide yes)
 			)
 		)
@@
 			)
 		)
-		(property "JLCPCB Part #" "C25744"
+		(property "LCSC Part #" "C25744"
 			(at 54.61 34.29 0)
 			(effects
@@
 					(size 1.27 1.27)
 				)
-				(hide yes)
 			)
 		)
@@
 			)
 		)
-		(property "JLCPCB Part #" "C307331 "
+		(property "LCSC Part #" "C307331 "
 			(at 156.21 55.88 0)
 			(effects
@@
 					(size 1.27 1.27)
 				)
-				(hide yes)
 			)
 		)
@@
 			)
 		)
-		(property "Value" "SIT8008xx-1x-xxE-100.000000"
+		(property "Value" "SITxxxxxx-1x-33E-50.000000"
 			(at 65.278 154.686 0)
 			(effects
@@
 			)
 		)
-		(property "JLCPCB Part #" "C1182928"
+		(property "LCSC Part #" "C1182928"
 			(at 43.18 158.75 0)
 			(effects
@@
 					(size 1.27 1.27)
 				)
-				(hide yes)
 			)
 		)
@@
 			)
 		)
-		(property "JLCPCB Part #" "C141836"
+		(property "LCSC Part #" "C141836"
 			(at 36.83 64.77 0)
 			(effects
@@
 					(size 1.27 1.27)
 				)
-				(hide yes)
 			)
 		)
@@
 			)
 		)
-		(property "JLCPCB Part #" "C25890 "
+		(property "LCSC Part #" "C25890 "
 			(at 54.61 111.76 0)
 			(effects
@@
 					(size 1.27 1.27)
 				)
-				(hide yes)
 			)
 		)
@@
 			)
 		)
-		(property "JLCPCB Part #" "C1043"
+		(property "LCSC Part #" "C1043"
 			(at 49.53 29.21 0)
 			(effects
@@
 					(size 1.27 1.27)
 				)
-				(hide yes)
 			)
 		)
@@
 			)
 		)
-		(property "JLCPCB Part #" "C59461 "
+		(property "LCSC Part #" "C59461 "
 			(at 24.13 67.31 0)
 			(effects
@@
 					(size 1.27 1.27)
 				)
-				(hide yes)
 			)
 		)
@@
 			)
 		)
-		(property "JLCPCB Part #" "C307331 "
+		(property "LCSC Part #" "C307331 "
 			(at 179.07 55.88 0)
 			(effects
@@
 					(size 1.27 1.27)
 				)
-				(hide yes)
 			)
 		)
@@
 			)
 		)
-		(property "JLCPCB Part #" "C307331 "
+		(property "LCSC Part #" "C307331 "
 			(at 213.36 55.88 0)
 			(effects
@@
 					(size 1.27 1.27)
 				)
-				(hide yes)
 			)
 		)
@@
 			)
 		)
-		(property "JLCPCB Part #" "C307331 "
+		(property "LCSC Part #" "C307331 "
 			(at 87.63 34.29 0)
 			(effects
@@
 					(size 1.27 1.27)
 				)
-				(hide yes)
 			)
 		)
@@
 			)
 		)
-		(property "JLCPCB Part #" ""
-			(at 63.5 101.6 0)
-			(effects
-				(font
-					(size 1.27 1.27)
-				)
-				(hide yes)
-			)
-		)
 		(pin "2"
 		)
@@
 			)
 		)
-		(property "JLCPCB Part #" "C307331 "
+		(property "LCSC Part #" "C307331 "
 			(at 201.93 55.88 0)
 			(effects
@@
 					(size 1.27 1.27)
 				)
-				(hide yes)
 			)
 		)
@@
 			)
 		)
-		(property "JLCPCB Part #" "C141836"
+		(property "LCSC Part #" "C141836"
 			(at 36.83 99.06 0)
 			(effects
@@
 					(size 1.27 1.27)
 				)
-				(hide yes)
 			)
 		)
@@
 			)
 		)
-		(property "JLCPCB Part #" "C59461 "
+		(property "LCSC Part #" "C59461 "
 			(at 24.13 101.6 0)
 			(effects
@@
 					(size 1.27 1.27)
 				)
-				(hide yes)
 			)
 		)
@@
 			)
 		)
-		(property "JLCPCB Part #" "C25756 "
+		(property "LCSC Part #" "C25756 "
 			(at 54.61 67.31 0)
 			(effects
@@
 					(size 1.27 1.27)
 				)
-				(hide yes)
 			)
 		)
@@
 			)
 		)
-		(property "JLCPCB Part #" "C1521614"
+		(property "LCSC Part #" "C1521614"
 			(at 240.03 73.66 0)
 			(effects
@@
 					(size 1.27 1.27)
 				)
-				(hide yes)
 			)
 		)
@@
 			)
 		)
-		(property "JLCPCB Part #" "C307331 "
+		(property "LCSC Part #" "C307331 "
 			(at 190.5 55.88 0)
 			(effects
@@
 					(size 1.27 1.27)
 				)
-				(hide yes)
 			)
 		)
@@
 			)
 		)
-		(property "JLCPCB Part #" "C307331 "
+		(property "LCSC Part #" "C307331 "
 			(at 167.64 55.88 0)
 			(effects
@@
 					(size 1.27 1.27)
 				)
-				(hide yes)
 			)
 		)
@@
 			)
 		)
-		(property "JLCPCB Part #" "C1043"
+		(property "LCSC Part #" "C1043"
 			(at 49.53 62.23 0)
 			(effects
@@
 					(size 1.27 1.27)
 				)
-				(hide yes)
 			)
 		)
@@
 			)
 		)
-		(property "JLCPCB Part #" "C307331 "
+		(property "LCSC Part #" "C307331 "
 			(at 27.94 160.02 0)
 			(effects
@@
 					(size 1.27 1.27)
 				)
-				(hide yes)
 			)
 		)
@@
 			)
 		)
-		(property "JLCPCB Part #" "C307331 "
+		(property "LCSC Part #" "C307331 "
 			(at 209.55 74.93 0)
 			(effects
@@
 					(size 1.27 1.27)
 				)
-				(hide yes)
 			)
 		)
@@
 			)
 		)
-		(property "JLCPCB Part #" "C59461 "
+		(property "LCSC Part #" "C59461 "
 			(at 63.5 34.29 0)
 			(effects
@@
 					(size 1.27 1.27)
 				)
-				(hide yes)
 			)
 		)
@@
 			)
 		)
-		(property "JLCPCB Part #" "C59461 "
+		(property "LCSC Part #" "C59461 "
 			(at 74.93 34.29 0)
 			(effects
@@
 					(size 1.27 1.27)
 				)
-				(hide yes)
 			)
 		)
@@
 			)
 		)
-		(property "JLCPCB Part #" "C307331 "
+		(property "LCSC Part #" "C307331 "
 			(at 76.2 101.6 0)
 			(effects
@@
 					(size 1.27 1.27)
 				)
-				(hide yes)
 			)
 		)
@@
 			)
 		)
-		(property "JLCPCB Part #" "C59461 "
+		(property "LCSC Part #" "C59461 "
 			(at 24.13 34.29 0)
 			(effects
@@
 					(size 1.27 1.27)
 				)
-				(hide yes)
 			)
 		)
@@
 			)
 		)
-		(property "JLCPCB Part #" "C25900 "
+		(property "LCSC Part #" "C25900 "
 			(at 54.61 77.47 0)
 			(effects
@@
 					(size 1.27 1.27)
 				)
-				(hide yes)
 			)
 		)
@@
 			)
 		)
-		(property "JLCPCB Part #" "C59461 "
+		(property "LCSC Part #" "C59461 "
 			(at 63.5 67.31 0)
 			(effects
@@
 					(size 1.27 1.27)
 				)
-				(hide yes)
 			)
 		)

Commit message: Last checks
Parts:
- C19: renamed from C15; LCSC Part # (none) -> C19702
- C23: renamed from C19; LCSC Part # (none) -> C19702
- C7: renamed from C4; LCSC Part # (none) -> C19702
- C8: renamed from C5; LCSC Part # (none) -> C19702
- C9: renamed from C6; LCSC Part # (none) -> C19702
- renumbered C7 to C10, C8 to C11, C9 to C12, C10 to C13, C11 to C14, C12 to C15, C13 to C16, C14 to C17, C51 to C18, C16 to C20, C17 to C21, C18 to C22, C52 to C24, C20 to C25, C1 to C3, C2 to C4, C3 to C5, C50 to C6, R9 to R10, R10 to R11, R5 to R6, R6 to R7, R7 to R8, R8 to R9, U3 to U1, U1 to U2, U2 to U3
