File: hardware/icepi-zero.kicad_pcb (KiCad board)
At the start: 4 copper layers, 65 x 30 mm, 134 parts, among them J1 Conn_02x20_Counter_Clockwise, J2 HDMI_C_1.3, J3 USB_C_Receptacle_USB2.0_14P, J4 USB_C_Receptacle_USB2.0_14P, J5 USB_C_Receptacle_USB2.0_14P, J6 Micro_SD_Card_Det2, SW1 SW_Push, U1 TLV62569DBV, U10 W9825G6KH, U11 W25Q128JVS, U2 TLV62569DBV, U3 ECP5U_12_CABGA256, U4 TLV62569DBV, U5 PCA9306DC1, U6 FT231XQ, U7 TPD2EUSB30A, U8 TPD2EUSB30A, U9 TPD2EUSB30A, Y1 SIT8008xx-1x-xxE-100.000000

Commit message: Final revision
Parts:
- Y1: value SIT8008xx-1x-xxE-100.000000 -> SITxxxxxx-1x-33E-50.000000
- moved TP9 0.09 mm to (157.8, 101.5)
- moved SW1 0.06 mm to (162.6, 102.4)
Connections:
- net Net-(U3B-PT27A/+/PCLKT0_1) renamed /ECP5/DBG1
- net Net-(U3C-PT35A/+/PCLKT1_0) renamed /ECP5/DBG2
Routing:
- net GND: track 77.6 -> 77.5 mm, vias 80 -> 87

Commit message: Last checks
Parts:
- added TP10: TestPoint, TestPoint:TestPoint_Pad_D1.0mm, B.Cu at (135.0, 117.1)
- added TP11: TestPoint, TestPoint:TestPoint_Pad_D1.0mm, B.Cu at (150.2, 115.2)
- added TP12: TestPoint, TestPoint:TestPoint_Pad_D1.0mm, B.Cu at (140.2, 116.8)
- added TP9: TestPoint, TestPoint:TestPoint_Pad_D1.0mm, B.Cu at (137.8, 116.8)
- moved C21 0.30 mm to (147.6, 103.5)
- moved C12 0.07 mm to (151.2, 105.1)
- moved C10 0.05 mm to (152.2, 103.5)
- moved C8 0.05 mm to (153.2, 105.1)
- moved C9 0.05 mm to (154.1, 103.1)
- renumbered C47 to C1, C7 to C10, C8 to C11, C9 to C12, C10 to C13, C11 to C14, C12 to C15, C13 to C16, C14 to C17, C51 to C18, C15 to C19, C48 to C2, C16 to C20, C17 to C21, C18 to C22, C19 to C23, C52 to C24, C20 to C25, C44 to C26, C45 to C27, C46 to C28, C21 to C29, C1 to C3, C22 to C30, C23 to C31, C24 to C32, C25 to C33, C26 to C34, C27 to C35, C28 to C36, C29 to C37, C49 to C38, C30 to C39, C2 to C4, C31 to C40, C32 to C41, C33 to C42, C34 to C43, C35 to C44, C36 to C45, C37 to C46, C38 to C47, C43 to C48, C40 to C49, C3 to C5, C41 to C50, C42 to C51, C39 to C52, C50 to C6, C4 to C7, C5 to C8, C6 to C9, D6 to D5, D5 to D6, R9 to R10, R10 to R11, R16 to R12, R17 to R13, R18 to R14, R11 to R15, R12 to R16, R13 to R17, R14 to R18, R15 to R19, R19 to R20, R20 to R21, R35 to R22, R36 to R23, R37 to R24, R38 to R25, R22 to R26, R24 to R27, R21 to R28, R23 to R29, R25 to R30, R26 to R31, R27 to R32, R28 to R33, R29 to R34, R30 to R35, R31 to R36, R32 to R37, R33 to R38, R34 to R5, R5 to R6, R6 to R7, R7 to R8, R8 to R9, TP4 to TP1, TP10 to TP13, TP9 to TP14, TP5 to TP2, TP1 to TP3, TP2 to TP4, TP6 to TP5, TP3 to TP6, U3 to U1, U1 to U2, U2 to U3
Connections:
- U6 pad 15: TXDEN -> unconnected-(U6-CBUS0-Pad15)
- U6 pad 16: ~{SLEEP} -> unconnected-(U6-CBUS3-Pad16)
- U6 pad 7: ~{TXLED} -> unconnected-(U6-CBUS2-Pad7)
Routing:
- net +3V3: track 96.7 -> 99.9 mm
- net JTAG_TCK: track 34.6 -> 37.8 mm
- net JTAG_TMS: track 33.3 -> 36.5 mm
- net GND: track 77.5 -> 80.5 mm, vias 87 -> 102
- net JTAG_TDI: track 31.8 -> 34.4 mm
- net JTAG_TDO: track 25.0 -> 27.5 mm
- net /ECP5/DBG1: track 5.77 -> 4.39 mm
Other:
- board text added: "Flash"
- board text added: "Icepi Zero v1.0"
- board text added: "USB1"
- board text added: "USB2"

Commit message: Final production files
Parts:
- H1, H2, H3, H4: footprint MountingHole:MountingHole_2.5mm -> MountingHole:MountingHole_2.7mm_M2.5
Routing:
- net GND: track 80.5 -> 83.1 mm
Changed lines of the file:
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@@
 	(net 250 "unconnected-(U1G-PL17D{slash}-{slash}LDQ20-PadJ5)")
 	(net 251 "unconnected-(U1E-PR29D{slash}-{slash}RDQ32-PadL12)")
-	(footprint "MountingHole:MountingHole_2.5mm"
+	(footprint "MountingHole:MountingHole_2.7mm_M2.5"
 		(layer "F.Cu")
 		(at 119.5 116.5)
-		(descr "Mounting Hole 2.5mm, no annular")
-		(tags "mounting hole 2.5mm no annular")
+		(descr "Mounting Hole 2.7mm, M2.5, no annular, generated by kicad-footprint-generator mountinghole.py")
+		(tags "mountinghole M2.5")
 		(property "Reference" "H3"
-			(at 0 -3.5 0)
+			(at 0 -3.65 0)
 			(layer "F.SilkS")
 			(hide yes)
@@
 		)
 		(property "Value" "MountingHole"
-			(at 0 3.5 0)
+			(at 0 3.65 0)
 			(layer "F.Fab")
 			(effects
@@
 		(property "Datasheet" ""
 			(at 0 0 0)
-			(unlocked yes)
 			(layer "F.Fab")
 			(hide yes)
@@
 		(property "Description" "Mounting Hole without connection"
 			(at 0 0 0)
-			(unlocked yes)
 			(layer "F.Fab")
 			(hide yes)
@@
 		(sheetname "/")
 		(sheetfile "icepi-zero.kicad_sch")
-		(solder_mask_margin 1.75)
-		(clearance 1.75)
+		(solder_mask_margin 1.5)
 		(attr exclude_from_pos_files exclude_from_bom dnp)
 		(fp_circle
 			(center 0 0)
-			(end 2.5 0)
+			(end 2.7 0)
 			(stroke
 				(width 0.15)
@@
 		(fp_circle
 			(center 0 0)
-			(end 2.75 0)
+			(end 2.95 0)
 			(stroke
 				(width 0.05)
@@
 		(pad "" np_thru_hole circle
 			(at 0 0)
-			(size 2.5 2.5)
-			(drill 2.5)
+			(size 2.7 2.7)
+			(drill 2.7)
 			(layers "*.Cu" "*.Mask")
 		)
@@
 		)
 	)
-	(footprint "MountingHole:MountingHole_2.5mm"
+	(footprint "MountingHole:MountingHole_2.7mm_M2.5"
 		(layer "F.Cu")
 		(at 119.5 93.5)
-		(descr "Mounting Hole 2.5mm, no annular")
-		(tags "mounting hole 2.5mm no annular")
+		(descr "Mounting Hole 2.7mm, M2.5, no annular, generated by kicad-footprint-generator mountinghole.py")
+		(tags "mountinghole M2.5")
 		(property "Reference" "H1"
-			(at 0 -3.5 0)
+			(at 0 -3.65 0)
 			(layer "F.SilkS")
 			(hide yes)
@@
 		)
 		(property "Value" "MountingHole"
-			(at 0 3.5 0)
+			(at 0 3.65 0)
 			(layer "F.Fab")
 			(effects
@@
 		(property "Datasheet" ""
 			(at 0 0 0)
-			(unlocked yes)
 			(layer "F.Fab")
 			(hide yes)
@@
 		(property "Description" "Mounting Hole without connection"
 			(at 0 0 0)
-			(unlocked yes)
 			(layer "F.Fab")
 			(hide yes)
@@
 		(sheetname "/")
 		(sheetfile "icepi-zero.kicad_sch")
-		(solder_mask_margin 1.75)
-		(clearance 1.75)
+		(solder_mask_margin 1.5)
 		(attr exclude_from_pos_files exclude_from_bom dnp)
 		(fp_circle
 			(center 0 0)
-			(end 2.5 0)
+			(end 2.7 0)
 			(stroke
 				(width 0.15)
@@
 		(fp_circle
 			(center 0 0)
-			(end 2.75 0)
+			(end 2.95 0)
 			(stroke
 				(width 0.05)
@@
 		(pad "" np_thru_hole circle
 			(at 0 0)
-			(size 2.5 2.5)
-			(drill 2.5)
+			(size 2.7 2.7)
+			(drill 2.7)
 			(layers "*.Cu" "*.Mask")
 		)
@@
 		)
 	)
-	(footprint "MountingHole:MountingHole_2.5mm"
+	(footprint "MountingHole:MountingHole_2.7mm_M2.5"
 		(layer "F.Cu")
 		(at 177.5 116.5)
-		(descr "Mounting Hole 2.5mm, no annular")
-		(tags "mounting hole 2.5mm no annular")
+		(descr "Mounting Hole 2.7mm, M2.5, no annular, generated by kicad-footprint-generator mountinghole.py")
+		(tags "mountinghole M2.5")
 		(property "Reference" "H4"
-			(at 0 -3.5 0)
+			(at 0 -3.65 0)
 			(layer "F.SilkS")
 			(hide yes)
@@
 		)
 		(property "Value" "MountingHole"
-			(at 0 3.5 0)
+			(at 0 3.65 0)
 			(layer "F.Fab")
 			(effects
@@
 		(property "Datasheet" ""
 			(at 0 0 0)
-			(unlocked yes)
 			(layer "F.Fab")
 			(hide yes)
@@
 		(property "Description" "Mounting Hole without connection"
 			(at 0 0 0)
-			(unlocked yes)
 			(layer "F.Fab")
 			(hide yes)
@@
 		(sheetname "/")
 		(sheetfile "icepi-zero.kicad_sch")
-		(solder_mask_margin 1.75)
-		(clearance 1.75)
+		(solder_mask_margin 1.5)
 		(attr exclude_from_pos_files exclude_from_bom dnp)
 		(fp_circle
 			(center 0 0)
-			(end 2.5 0)
+			(end 2.7 0)
 			(stroke
 				(width 0.15)
@@
 		(fp_circle
 			(center 0 0)
-			(end 2.75 0)
+			(end 2.95 0)
 			(stroke
 				(width 0.05)
@@
 		(pad "" np_thru_hole circle
 			(at 0 0)
-			(size 2.5 2.5)
-			(drill 2.5)
+			(size 2.7 2.7)
+			(drill 2.7)
 			(layers "*.Cu" "*.Mask")
 		)
@@
 		)
 	)
-	(footprint "MountingHole:MountingHole_2.5mm"
+	(footprint "MountingHole:MountingHole_2.7mm_M2.5"
 		(layer "F.Cu")
 		(at 177.5 93.5)
-		(descr "Mounting Hole 2.5mm, no annular")
-		(tags "mounting hole 2.5mm no annular")
+		(descr "Mounting Hole 2.7mm, M2.5, no annular, generated by kicad-footprint-generator mountinghole.py")
+		(tags "mountinghole M2.5")
 		(property "Reference" "H2"
-			(at 0 -3.5 0)
+			(at 0 -3.65 0)
 			(layer "F.SilkS")
 			(hide yes)
@@
 		)
 		(property "Value" "MountingHole"
-			(at 0 3.5 0)
+			(at 0 3.65 0)
 			(layer "F.Fab")
 			(effects
@@
 		(property "Datasheet" ""
 			(at 0 0 0)
-			(unlocked yes)
 			(layer "F.Fab")
 			(hide yes)
@@
 		(property "Description" "Mounting Hole without connection"
 			(at 0 0 0)
-			(unlocked yes)
 			(layer "F.Fab")
 			(hide yes)
@@
 		(sheetname "/")
 		(sheetfile "icepi-zero.kicad_sch")
-		(solder_mask_margin 1.75)
-		(clearance 1.75)
+		(solder_mask_margin 1.5)
 		(attr exclude_from_pos_files exclude_from_bom dnp)
 		(fp_circle
 			(center 0 0)
-			(end 2.5 0)
+			(end 2.7 0)
 			(stroke
 				(width 0.15)
@@
 		(fp_circle
 			(center 0 0)
-			(end 2.75 0)
+			(end 2.95 0)
 			(stroke
 				(width 0.05)
@@
 		(pad "" np_thru_hole circle
 			(at 0 0)
-			(size 2.5 2.5)
-			(drill 2.5)
+			(size 2.7 2.7)
+			(drill 2.7)
 			(layers "*.Cu" "*.Mask")
 		)
@@
 		(sheetname "/USB/")
 		(sheetfile "usb.kicad_sch")
-		(attr exclude_from_pos_files)
+		(attr exclude_from_pos_files dnp)
 		(fp_circle
 			(center 0 0)
@@
 		(sheetname "/USB/")
 		(sheetfile "usb.kicad_sch")
-		(attr exclude_from_pos_files)
+		(attr exclude_from_pos_files dnp)
 		(fp_circle
 			(center 0 0)
@@
 		(sheetname "/USB/")
 		(sheetfile "usb.kicad_sch")
-		(attr exclude_from_pos_files)
+		(attr exclude_from_pos_files dnp)
 		(fp_circle
 			(center 0 0)
@@
 		(sheetname "/USB/")
 		(sheetfile "usb.kicad_sch")
-		(attr exclude_from_pos_files)
+		(attr exclude_from_pos_files dnp)
 		(fp_circle
 			(center 0 0)
@@
 	)
 	(segment
+		(start 146.786 110.909887)
+		(end 146.786 111.139)
+		(width 0.17)
+		(layer "F.Cu")
+		(net 38)
+	)
+	(segment
 		(start 168.71 111.97)
 		(end 168.445 111.97)
@@
 	)
 	(segment
+		(start 146.786 110.336)
+		(end 146.786 110.909887)
+		(width 0.17)
+		(layer "F.Cu")
+		(net 38)
+	)
+	(segment
 		(start 143.98 107.57)
 		(end 144 107.55)
@@
 	)
 	(segment
+		(start 146.4 109.95)
+		(end 146.786 110.336)
+		(width 0.17)
+		(layer "F.Cu")
+		(net 38)
+	)
+	(segment
 		(start 129.54 100.71)
 		(end 129.54 101.225)
@@
 		(layer "F.Cu")
 		(net 38)
+	)
+	(segment
+		(start 146.15 111.275)
+		(end 145.225 112.2)
+		(width 0.3)
+		(layer "F.Cu")
+		(net 38)
