File: hardware/usb.kicad_sch (KiCad schematic)
At the start: 27 parts, among them J3 USB_C_Receptacle_USB2.0_14P, J4 USB_C_Receptacle_USB2.0_14P, J5 USB_C_Receptacle_USB2.0_14P, U1 ECP5U_12_CABGA256, U6 FT231XQ, U7 TPD2EUSB30A, U8 TPD2EUSB30A, U9 TPD2EUSB30A

Commit message: Final production files
Parts:
- TP10, TP11, TP12, TP9: now not fitted
Changed lines of the file:
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@@
 		(in_bom yes)
 		(on_board yes)
-		(dnp no)
+		(dnp yes)
 		(fields_autoplaced yes)
 		(property "Reference" "TP10"
@@
 		(in_bom yes)
 		(on_board yes)
-		(dnp no)
+		(dnp yes)
 		(fields_autoplaced yes)
 		(property "Reference" "TP11"
@@
 		(in_bom yes)
 		(on_board yes)
-		(dnp no)
+		(dnp yes)
 		(fields_autoplaced yes)
 		(property "Reference" "TP12"
@@
 		(in_bom yes)
 		(on_board yes)
-		(dnp no)
+		(dnp yes)
 		(fields_autoplaced yes)
 		(property "Reference" "TP9"
