File: hardware/v1.0/ecp5.kicad_sch (KiCad schematic)
At the start: 8 parts, among them U1 ECP5U_12_CABGA256

Commit message: Finish lpf
Connections:
- net SW2: no longer names the net of U1.C5 (PT15A/+)
- no-connect marks 50 -> 51
Changed lines of the file:
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@@
+	)
+	(no_connect
+		(at 38.1 55.88)
 	)
 	(no_connect
@@
 			(effects
 				(font
-					(size 1.27 1.27)
-				)
-				(justify right)
-				(hide yes)
-			)
-		)
-	)
-	(global_label "SW2"
-		(shape input)
-		(at 38.1 55.88 180)
-		(fields_autoplaced yes)
-		(effects
-			(font
-				(size 1.27 1.27)
-			)
-			(justify right)
-		)
-		(property "Intersheetrefs" "${INTERSHEET_REFS}"
-			(at 31.2444 55.88 0)
-			(effects
-				(font
