File: hardware/v1.0/power.kicad_sch (KiCad schematic)
At the start: 38 parts, among them U1 ECP5U_12_CABGA256, U2 TLV62569DBV, U3 TLV62569DBV, U4 TLV62569DBV, Y1 SITxxxxxx-1x-33E-50.000000

Commit message: Finish lpf
Other:
- note added: "50MHz Clock"
- note removed: "40MHz Clock"
Changed lines of the file:
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@@
 		)
 	)
-	(text "40MHz Clock"
+	(text "50MHz Clock"
 		(exclude_from_sim no)
 		(at 43.688 140.97 0)
